Commit message: more accurate joint locations

File: predator_description/urdf/predator.xacro (robot description, xacro)
@@ -3,7 +3,7 @@
     <link name="base_link">
         <visual>
-            <origin rpy="0 0 0" xyz="0 0 0"/>
+            <origin rpy="0 0 0" xyz="0 0 0.02262"/>
             <geometry>
-                <box size="1 1 1"/>
+                <box size="0.197 0.197 0.04524"/>
             </geometry>
         </visual>
@@ -12,5 +12,5 @@
         <axis xyz="0 0 1" />
         <limit effort="1000.0" lower="-3.14" upper="3.14" velocity="0.5" />
-        <origin rpy="0 0 0" xyz="0 0 0.5"/>
+        <origin rpy="0 0 0" xyz="0 0 0.203"/>
         <parent link="base_link"/>
         <child link="link1"/>
@@ -18,13 +18,13 @@
     <link name="link1">
         <visual>
-            <origin rpy="0 0 0" xyz="0 0 0.2"/>
+            <origin rpy="0 0 0" xyz="0 0 -0.07888"/>
             <geometry>
-                <cylinder radius="0.35" length="0.4"/>
+                <cylinder radius="0.0985" length="0.15776"/>
             </geometry>
         </visual>
         <visual>
-            <origin rpy="1.8 0 0" xyz="0 0.5 0.3"/>
+            <origin rpy="1.57079632679 0 0" xyz="0 0.07 0"/>
             <geometry>
-                <cylinder radius="0.1" length="1"/>
+                <cylinder radius="0.02" length="0.130"/>
             </geometry>
         </visual>
@@ -33,5 +33,5 @@
         <axis xyz="1 0 0" />
         <limit effort="1000.0" lower="-3.14" upper="3.14" velocity="0.5" />
-        <origin rpy="0 0 0" xyz="0 0.9 0.5"/>
+        <origin rpy="0 0 0" xyz="0 0.1295 0"/>
         <parent link="link1"/>
         <child link="link2"/>
@@ -39,7 +39,7 @@
     <link name="link2">
         <visual>
-            <origin rpy="3.14 0 0" xyz="0 0 0.5 "/>
+            <origin rpy="3.14 0 0" xyz="0 0 0.4375"/>
             <geometry>
-                <cylinder radius="0.1" length="1"/>
+                <cylinder radius="0.0889" length="0.875"/>
             </geometry>
         </visual>
@@ -48,5 +48,5 @@
         <axis xyz="1 0 0" />
         <limit effort="1000.0" lower="-3.14" upper="3.14" velocity="0.5" />
-        <origin rpy="0 0 0" xyz="0 0 1"/>
+        <origin rpy="0 0 0" xyz="0 0 0.875"/>
         <parent link="link2"/>
         <child link="link3"/>
@@ -54,7 +54,13 @@
     <link name="link3">
         <visual>
-            <origin rpy="-2.6 0 0" xyz="0 0.35 -0.35"/>
+            <origin rpy="1.57079632679 0 0" xyz="0 0.15 0"/>
             <geometry>
-                <cylinder radius="0.1" length="1"/>
+                <cylinder radius="0.0889" length="0.3"/>
+            </geometry>
+        </visual>
+        <visual>
+            <origin rpy="0 0 0" xyz="0 0.1278 -0.274"/>
+            <geometry>
+                <cylinder radius="0.05" length="0.548"/>
             </geometry>
         </visual>
@@ -63,5 +69,5 @@
         <axis xyz="1 0 0" />
         <limit effort="1000.0" lower="-3.14" upper="3.14" velocity="0.5" />
-        <origin rpy="0 0 0" xyz="0 0.685 -0.8"/>
+        <origin rpy="0 0 0" xyz="0 0.1389 -0.548"/>
         <parent link="link3"/>
         <child link="link4"/>
@@ -69,14 +75,14 @@
     <link name="link4">
         <visual>
-            <origin rpy="1.571 0 0" xyz="0 0.25 0"/>
+            <origin rpy="0 0 0" xyz="0 0 -0.0605"/>
             <geometry>
-                <cylinder radius="0.1" length="0.5"/>
+                <cylinder radius="0.02" length="0.121"/>
             </geometry>
         </visual>
     </link>
     <joint name="link_04__link_05" type="revolute">
-        <axis xyz="0 0 1" />
+        <axis xyz="0 1 0" />
         <limit effort="1000.0" lower="-3.14" upper="3.14" velocity="0.5" />
-        <origin rpy="0 0 0" xyz="0 0.6 0"/>
+        <origin rpy="0 0 0" xyz="0 0 -0.121"/>
         <parent link="link4"/>
         <child link="link5"/>
@@ -84,7 +90,7 @@
     <link name="link5">
         <visual>
-            <origin rpy="1.571 0 0" xyz="0 0.25 0"/>
+            <origin rpy="0 0 0" xyz="0 0 -0.05"/>
             <geometry>
-                <cylinder radius="0.1" length="0.5"/>
+                <cylinder radius="0.01" length="0.1"/>
             </geometry>
         </visual>

Commit message: added a parameter file and fixed joint limits

File: predator_description/urdf/predator.xacro (robot description, xacro)
@@ -1,9 +1,10 @@
 <?xml version="1.0"?>
 <robot name="mrm" xmlns:xacro="http://www.ros.org/wiki/xacro">
+    <xacro:include filename="$(find predator_description)/urdf/robot_parameter.xacro" />
     <link name="base_link">
         <visual>
-            <origin rpy="0 0 0" xyz="0 0 0.02262"/>
+            <origin rpy="0 0 0" xyz="0 0 ${base_height/2}"/>
             <geometry>
-                <box size="0.197 0.197 0.04524"/>
+                <box size="${base_width} ${base_width} ${base_height}"/>
             </geometry>
         </visual>
@@ -11,6 +12,6 @@
     <joint name="base_link__link_01" type="revolute">
         <axis xyz="0 0 1" />
-        <limit effort="1000.0" lower="-3.14" upper="3.14" velocity="0.5" />
-        <origin rpy="0 0 0" xyz="0 0 0.203"/>
+        <limit effort="1000.0" lower="${-3/4*pi}" upper="${3/4*pi}" velocity="0.5" />
+        <origin rpy="0 0 0" xyz="${joint1}"/>
         <parent link="base_link"/>
         <child link="link1"/>
@@ -18,11 +19,11 @@
     <link name="link1">
         <visual>
-            <origin rpy="0 0 0" xyz="0 0 -0.07888"/>
+            <origin rpy="0 0 0" xyz="0 0 ${link1_length/-2}"/>
             <geometry>
-                <cylinder radius="0.0985" length="0.15776"/>
+                <cylinder radius="0.0985" length="${link1_length}"/>
             </geometry>
         </visual>
         <visual>
-            <origin rpy="1.57079632679 0 0" xyz="0 0.07 0"/>
+            <origin rpy="${pi/2} 0 0" xyz="0 0.07 0"/>
             <geometry>
                 <cylinder radius="0.02" length="0.130"/>
@@ -32,5 +33,5 @@
     <joint name="link_01__link_02" type="revolute">
         <axis xyz="1 0 0" />
-        <limit effort="1000.0" lower="-3.14" upper="3.14" velocity="0.5" />
+        <limit effort="1000.0" lower="${-pi*2/3}" upper="0" velocity="0.5" />
         <origin rpy="0 0 0" xyz="0 0.1295 0"/>
         <parent link="link1"/>
@@ -47,5 +48,5 @@
     <joint name="link_02__link_03" type="revolute">
         <axis xyz="1 0 0" />
-        <limit effort="1000.0" lower="-3.14" upper="3.14" velocity="0.5" />
+        <limit effort="1000.0" lower="0" upper="${125/180.0*pi}" velocity="0.5" />
         <origin rpy="0 0 0" xyz="0 0 0.875"/>
         <parent link="link2"/>
@@ -68,5 +69,5 @@
     <joint name="link_03__link_04" type="revolute">
         <axis xyz="1 0 0" />
-        <limit effort="1000.0" lower="-3.14" upper="3.14" velocity="0.5" />
+        <limit effort="1000.0" lower="${-100/180*pi}" upper="${100/180*pi}" velocity="0.5" />
         <origin rpy="0 0 0" xyz="0 0.1389 -0.548"/>
         <parent link="link3"/>
@@ -83,5 +84,5 @@
     <joint name="link_04__link_05" type="revolute">
         <axis xyz="0 1 0" />
-        <limit effort="1000.0" lower="-3.14" upper="3.14" velocity="0.5" />
+        <limit effort="1000.0" lower="${-100/180*pi}" upper="${100/180*pi}" velocity="0.5" />
         <origin rpy="0 0 0" xyz="0 0 -0.121"/>
         <parent link="link4"/>

Commit message: added joint macro + added inertia and collisions

File: predator_description/urdf/predator.xacro (robot description, xacro)
@@ -2,4 +2,5 @@
 <robot name="mrm" xmlns:xacro="http://www.ros.org/wiki/xacro">
     <xacro:include filename="$(find predator_description)/urdf/robot_parameter.xacro" />
+    <xacro:include filename="$(find predator_description)/urdf/links_joints.xacro" />
     <link name="base_link">
         <visual>
@@ -9,12 +10,19 @@
             </geometry>
         </visual>
+        <collision>
+            <origin rpy="0 0 0" xyz="0 0 ${base_height/2}"/>
+            <geometry>
+                <box size="${base_width} ${base_width} ${base_height}"/>
+            </geometry>
+        </collision>
+        <inertial>
+            <mass value="10"/>
+            <inertia ixx="0.4" ixy="0.0" ixz="0.0"
+                     iyy="0.4" iyz="0.0"
+                     izz="0.2"/>
+            <origin rpy="0 0 0" xyz="0 0 ${base_height/2}"/>
+        </inertial>
     </link>
-    <joint name="base_link__link_01" type="revolute">
-        <axis xyz="0 0 1" />
-        <limit effort="1000.0" lower="${-3/4*pi}" upper="${3/4*pi}" velocity="0.5" />
-        <origin rpy="0 0 0" xyz="${joint1}"/>
-        <parent link="base_link"/>
-        <child link="link1"/>
-    </joint>
+    <revolute_joint name="azimuth_joint" />
     <link name="link1">
         <visual>
@@ -24,4 +32,17 @@
             </geometry>
         </visual>
+        <collision>
+            <origin rpy="0 0 0" xyz="0 0 ${link1_length/-2}"/>
+            <geometry>
+                <cylinder radius="0.0985" length="${link1_length}"/>
+            </geometry>
+        </collision>
+        <inertial>
+            <mass value="10"/>
+            <inertia ixx="0.4" ixy="0.0" ixz="0.0"
+                     iyy="0.4" iyz="0.0"
+                     izz="0.2"/>
+            <origin rpy="0 0 0" xyz="0 0 ${link1_length/-2}"/>
+        </inertial>
         <visual>
             <origin rpy="${pi/2} 0 0" xyz="0 0.07 0"/>
@@ -30,9 +51,15 @@
             </geometry>
         </visual>
+        <collision>
+            <origin rpy="${pi/2} 0 0" xyz="0 0.07 0"/>
+            <geometry>
+                <cylinder radius="0.02" length="0.130"/>
+            </geometry>
+        </collision>
     </link>
-    <joint name="link_01__link_02" type="revolute">
-        <axis xyz="1 0 0" />
-        <limit effort="1000.0" lower="${-pi*2/3}" upper="0" velocity="0.5" />
-        <origin rpy="0 0 0" xyz="0 0.1295 0"/>
+    <joint name="elevation" type="revolute">
+        <axis xyz="-1 0 0" />
+        <limit effort="1000.0" lower="0" upper="${pi*2/3}" velocity="0.5" />
+        <origin rpy="0 0 0" xyz="${elevation_joint_location}"/>
         <parent link="link1"/>
         <child link="link2"/>
@@ -45,4 +72,17 @@
             </geometry>
         </visual>
+        <collision>
+            <origin rpy="3.14 0 0" xyz="0 0 0.4375"/>
+            <geometry>
+                <cylinder radius="0.0889" length="0.875"/>
+            </geometry>
+        </collision>
+        <inertial>
+            <mass value="10"/>
+            <inertia ixx="0.4" ixy="0.0" ixz="0.0"
+                     iyy="0.4" iyz="0.0"
+                     izz="0.2"/>
+            <origin rpy="3.14 0 0" xyz="0 0 0.4375"/>
+        </inertial>
     </link>
     <joint name="link_02__link_03" type="revolute">
@@ -60,4 +100,10 @@
             </geometry>
         </visual>
+        <collision>
+            <origin rpy="1.57079632679 0 0" xyz="0 0.15 0"/>
+            <geometry>
+                <cylinder radius="0.0889" length="0.3"/>
+            </geometry>
+        </collision>
         <visual>
             <origin rpy="0 0 0" xyz="0 0.1278 -0.274"/>
@@ -66,4 +112,17 @@
             </geometry>
         </visual>
+        <collision>
+            <origin rpy="0 0 0" xyz="0 0.1278 -0.274"/>
+            <geometry>
+                <cylinder radius="0.05" length="0.548"/>
+            </geometry>
+        </collision>
+        <inertial>
+            <mass value="10"/>
+            <inertia ixx="0.4" ixy="0.0" ixz="0.0"
+                     iyy="0.4" iyz="0.0"
+                     izz="0.2"/>
+            <origin rpy="0 0 0" xyz="0 0.1278 -0.274"/>
+        </inertial>
     </link>
     <joint name="link_03__link_04" type="revolute">
@@ -81,4 +140,17 @@
             </geometry>
         </visual>
+        <collision>
+            <origin rpy="0 0 0" xyz="0 0 -0.0605"/>
+            <geometry>
+                <cylinder radius="0.02" length="0.121"/>
+            </geometry>
+        </collision>
+        <inertial>
+            <mass value="10"/>
+            <inertia ixx="0.4" ixy="0.0" ixz="0.0"
+                     iyy="0.4" iyz="0.0"
+                     izz="0.2"/>
+            <origin rpy="0 0 0" xyz="0 0 -0.0605"/>
+        </inertial>
     </link>
     <joint name="link_04__link_05" type="revolute">
@@ -96,4 +168,17 @@
             </geometry>
         </visual>
+        <collision>
+            <origin rpy="0 0 0" xyz="0 0 -0.05"/>
+            <geometry>
+                <cylinder radius="0.01" length="0.1"/>
+            </geometry>
+        </collision>
+        <inertial>
+            <mass value="10"/>
+            <inertia ixx="0.4" ixy="0.0" ixz="0.0"
+                     iyy="0.4" iyz="0.0"
+                     izz="0.2"/>
+            <origin rpy="0 0 0" xyz="0 0 -0.05"/>
+        </inertial>
     </link>
 </robot>

File: predator_description/urdf/robot_parameter.xacro (robot description, xacro)
@@ -7,6 +7,8 @@
   <xacro:property name="base_width" value="0.197"/>
   <xacro:property name="base_height" value="0.04524" />
-  <!-- Joint 1 location (top of the first cylinder) -->
+  <!-- azimuth joint -->
   <xacro:property name="joint1" value="0 0 0.203"/>
+  <!-- elevation joint -->
+  <xacro:property name="elevation_joint_location" value="0 0.1295 0"/>
   <!-- Link1 -->
   <xacro:property name="link1_length" value="0.15776"/>

Commit message: added transmission links and disables self collision

File: predator_description/urdf/predator.xacro (robot description, xacro)
@@ -24,5 +24,18 @@
         </inertial>
     </link>
+    <gazebo reference="base_link">
+        <selfCollide>false</selfCollide>
+    </gazebo>
     <revolute_joint name="azimuth_joint" />
+    <transmission name="azimuth_trans">
+        <type>transmission_interface/SimpleTransmission</type>
+        <joint name="azimuth_joint">
+            <hardwareInterface>hardware_interface/EffortJointInterface</hardwareInterface>
+        </joint>
+        <actuator name="azimuth_motor">
+            <mechanicalReduction>1</mechanicalReduction>
+            <hardwareInterface>hardware_interface/EffortJointInterface</hardwareInterface>
+        </actuator>
+    </transmission>
     <link name="link1">
         <visual>
@@ -39,5 +52,5 @@
         </collision>
         <inertial>
-            <mass value="10"/>
+            <mass value="1"/>
             <inertia ixx="0.4" ixy="0.0" ixz="0.0"
                      iyy="0.4" iyz="0.0"
@@ -58,5 +71,8 @@
         </collision>
     </link>
-    <joint name="elevation" type="revolute">
+    <gazebo reference="link1">
+        <selfCollide>false</selfCollide>
+    </gazebo>
+    <joint name="elevation_joint" type="revolute">
         <axis xyz="-1 0 0" />
         <limit effort="1000.0" lower="0" upper="${pi*2/3}" velocity="0.5" />
@@ -65,4 +81,14 @@
         <child link="link2"/>
     </joint>
+    <transmission name="elevation_trans">
+        <type>transmission_interface/SimpleTransmission</type>
+        <joint name="elevation_joint">
+            <hardwareInterface>hardware_interface/EffortJointInterface</hardwareInterface>
+        </joint>
+        <actuator name="elevation_motor">
+            <mechanicalReduction>1</mechanicalReduction>
+            <hardwareInterface>hardware_interface/EffortJointInterface</hardwareInterface>
+        </actuator>
+    </transmission>
     <link name="link2">
         <visual>
@@ -79,5 +105,5 @@
         </collision>
         <inertial>
-            <mass value="10"/>
+            <mass value="1"/>
             <inertia ixx="0.4" ixy="0.0" ixz="0.0"
                      iyy="0.4" iyz="0.0"
@@ -86,5 +112,8 @@
         </inertial>
     </link>
-    <joint name="link_02__link_03" type="revolute">
+    <gazebo reference="link2">
+        <selfCollide>false</selfCollide>
+    </gazebo>
+    <joint name="link_02__link_03_joint" type="revolute">
         <axis xyz="1 0 0" />
         <limit effort="1000.0" lower="0" upper="${125/180.0*pi}" velocity="0.5" />
@@ -93,4 +122,14 @@
         <child link="link3"/>
     </joint>
+    <transmission name="link_02__link_03_trans">
+        <type>transmission_interface/SimpleTransmission</type>
+        <joint name="link_02__link_03_joint">
+            <hardwareInterface>hardware_interface/EffortJointInterface</hardwareInterface>
+        </joint>
+        <actuator name="link_02__link_03_motor">
+            <mechanicalReduction>1</mechanicalReduction>
+            <hardwareInterface>hardware_interface/EffortJointInterface</hardwareInterface>
+        </actuator>
+    </transmission>
     <link name="link3">
         <visual>
@@ -119,5 +158,5 @@
         </collision>
         <inertial>
-            <mass value="10"/>
+            <mass value=".1"/>
             <inertia ixx="0.4" ixy="0.0" ixz="0.0"
                      iyy="0.4" iyz="0.0"
@@ -126,5 +165,8 @@
         </inertial>
     </link>
-    <joint name="link_03__link_04" type="revolute">
+    <gazebo reference="link3">
+        <selfCollide>false</selfCollide>
+    </gazebo>
+    <joint name="link_03__link_04_joint" type="revolute">
         <axis xyz="1 0 0" />
         <limit effort="1000.0" lower="${-100/180*pi}" upper="${100/180*pi}" velocity="0.5" />
@@ -133,4 +175,14 @@
         <child link="link4"/>
     </joint>
+    <transmission name="link_03__link_04_trans">
+        <type>transmission_interface/SimpleTransmission</type>
+        <joint name="link_03__link_04_joint">
+            <hardwareInterface>hardware_interface/EffortJointInterface</hardwareInterface>
+        </joint>
+        <actuator name="link_03__link_04_motor">
+            <mechanicalReduction>1</mechanicalReduction>
+            <hardwareInterface>hardware_interface/EffortJointInterface</hardwareInterface>
+        </actuator>
+    </transmission>
     <link name="link4">
         <visual>
@@ -147,5 +199,5 @@
         </collision>
         <inertial>
-            <mass value="10"/>
+            <mass value=".1"/>
             <inertia ixx="0.4" ixy="0.0" ixz="0.0"
                      iyy="0.4" iyz="0.0"
@@ -154,5 +206,8 @@
         </inertial>
     </link>
-    <joint name="link_04__link_05" type="revolute">
+    <gazebo reference="link4">
+        <selfCollide>false</selfCollide>
+    </gazebo>
+    <joint name="link_04__link_05_joint" type="revolute">
         <axis xyz="0 1 0" />
         <limit effort="1000.0" lower="${-100/180*pi}" upper="${100/180*pi}" velocity="0.5" />
@@ -161,4 +216,14 @@
         <child link="link5"/>
     </joint>
+    <transmission name="link_04__link_05_trans">
+        <type>transmission_interface/SimpleTransmission</type>
+        <joint name="link_04__link_05_joint">
+            <hardwareInterface>hardware_interface/EffortJointInterface</hardwareInterface>
+        </joint>
+        <actuator name="link_04__link_05_motor">
+            <mechanicalReduction>1</mechanicalReduction>
+            <hardwareInterface>hardware_interface/EffortJointInterface</hardwareInterface>
+        </actuator>
+    </transmission>
     <link name="link5">
         <visual>
@@ -175,5 +240,5 @@
         </collision>
         <inertial>
-            <mass value="10"/>
+            <mass value=".1"/>
             <inertia ixx="0.4" ixy="0.0" ixz="0.0"
                      iyy="0.4" iyz="0.0"
@@ -182,3 +247,10 @@
         </inertial>
     </link>
+    <gazebo reference="link5">
+        <selfCollide>false</selfCollide>
+    </gazebo>
+    <gazebo>
+      <plugin name="gazebo_ros_control" filename="libgazebo_ros_control.so">
+    </plugin>
+  </gazebo>
 </robot>
