Commit message: Rename joints to manufacturer's convention

File: predator_description/urdf/predator.xacro (robot description, xacro)
@@ -27,11 +27,11 @@
         <selfCollide>false</selfCollide>
     </gazebo>
-    <revolute_joint name="azimuth_joint" />
-    <transmission name="azimuth_trans">
-        <type>transmission_interface/SimpleTransmission</type>
-        <joint name="azimuth_joint">
-            <hardwareInterface>hardware_interface/EffortJointInterface</hardwareInterface>
-        </joint>
-        <actuator name="azimuth_motor">
+    <revolute_joint name="shoulder_azimuth_joint" />
+    <transmission name="shoulder_azimuth_trans">
+        <type>transmission_interface/SimpleTransmission</type>
+        <joint name="shoulder_azimuth_joint">
+            <hardwareInterface>hardware_interface/EffortJointInterface</hardwareInterface>
+        </joint>
+        <actuator name="shoulder_azimuth_motor">
             <mechanicalReduction>1</mechanicalReduction>
             <hardwareInterface>hardware_interface/EffortJointInterface</hardwareInterface>
@@ -74,5 +74,5 @@
         <selfCollide>false</selfCollide>
     </gazebo>
-    <joint name="elevation_joint" type="revolute">
+    <joint name="shoulder_elevation_joint" type="revolute">
         <axis xyz="-1 0 0" />
         <limit effort="1000.0" lower="0" upper="${pi*2/3}" velocity="0.5" />
@@ -81,10 +81,10 @@
         <child link="link2"/>
     </joint>
-    <transmission name="elevation_trans">
-        <type>transmission_interface/SimpleTransmission</type>
-        <joint name="elevation_joint">
-            <hardwareInterface>hardware_interface/EffortJointInterface</hardwareInterface>
-        </joint>
-        <actuator name="elevation_motor">
+    <transmission name="shoulder_elevation_trans">
+        <type>transmission_interface/SimpleTransmission</type>
+        <joint name="shoulder_elevation_joint">
+            <hardwareInterface>hardware_interface/EffortJointInterface</hardwareInterface>
+        </joint>
+        <actuator name="shoulder_elevation_motor">
             <mechanicalReduction>1</mechanicalReduction>
             <hardwareInterface>hardware_interface/EffortJointInterface</hardwareInterface>
@@ -115,5 +115,5 @@
         <selfCollide>false</selfCollide>
     </gazebo>
-    <joint name="link_02__link_03_joint" type="revolute">
+    <joint name="elbow_pivot_joint" type="revolute">
         <axis xyz="1 0 0" />
         <limit effort="1000.0" lower="0" upper="${125/180.0*pi}" velocity="0.5" />
@@ -122,10 +122,10 @@
         <child link="link3"/>
     </joint>
-    <transmission name="link_02__link_03_trans">
-        <type>transmission_interface/SimpleTransmission</type>
-        <joint name="link_02__link_03_joint">
-            <hardwareInterface>hardware_interface/EffortJointInterface</hardwareInterface>
-        </joint>
-        <actuator name="link_02__link_03_motor">
+    <transmission name="elbow_pivot_trans">
+        <type>transmission_interface/SimpleTransmission</type>
+        <joint name="elbow_pivot_joint">
+            <hardwareInterface>hardware_interface/EffortJointInterface</hardwareInterface>
+        </joint>
+        <actuator name="elbow_pivot_motor">
             <mechanicalReduction>1</mechanicalReduction>
             <hardwareInterface>hardware_interface/EffortJointInterface</hardwareInterface>
@@ -168,5 +168,5 @@
         <selfCollide>false</selfCollide>
     </gazebo>
-    <joint name="link_03__link_04_joint" type="revolute">
+    <joint name="wrist_pitch_joint" type="revolute">
         <axis xyz="1 0 0" />
         <limit effort="1000.0" lower="${-100/180*pi}" upper="${100/180*pi}" velocity="0.5" />
@@ -175,10 +175,10 @@
         <child link="link4"/>
     </joint>
-    <transmission name="link_03__link_04_trans">
-        <type>transmission_interface/SimpleTransmission</type>
-        <joint name="link_03__link_04_joint">
-            <hardwareInterface>hardware_interface/EffortJointInterface</hardwareInterface>
-        </joint>
-        <actuator name="link_03__link_04_motor">
+    <transmission name="wrist_pitch_trans">
+        <type>transmission_interface/SimpleTransmission</type>
+        <joint name="wrist_pitch_joint">
+            <hardwareInterface>hardware_interface/EffortJointInterface</hardwareInterface>
+        </joint>
+        <actuator name="wrist_pitch_motor">
             <mechanicalReduction>1</mechanicalReduction>
             <hardwareInterface>hardware_interface/EffortJointInterface</hardwareInterface>
@@ -209,5 +209,5 @@
         <selfCollide>false</selfCollide>
     </gazebo>
-    <joint name="link_04__link_05_joint" type="revolute">
+    <joint name="wrist_yaw_joint" type="revolute">
         <axis xyz="0 1 0" />
         <limit effort="1000.0" lower="${-100/180*pi}" upper="${100/180*pi}" velocity="0.5" />
@@ -216,10 +216,10 @@
         <child link="link5"/>
     </joint>
-    <transmission name="link_04__link_05_trans">
-        <type>transmission_interface/SimpleTransmission</type>
-        <joint name="link_04__link_05_joint">
-            <hardwareInterface>hardware_interface/EffortJointInterface</hardwareInterface>
-        </joint>
-        <actuator name="link_04__link_05_motor">
+    <transmission name="wrist_yaw_trans">
+        <type>transmission_interface/SimpleTransmission</type>
+        <joint name="wrist_yaw_joint">
+            <hardwareInterface>hardware_interface/EffortJointInterface</hardwareInterface>
+        </joint>
+        <actuator name="wrist_yaw_motor">
             <mechanicalReduction>1</mechanicalReduction>
             <hardwareInterface>hardware_interface/EffortJointInterface</hardwareInterface>

Commit message: Make links look better

File: predator_description/urdf/predator.xacro (robot description, xacro)
@@ -95,5 +95,5 @@
             <origin rpy="3.14 0 0" xyz="0 0 0.4375"/>
             <geometry>
-                <cylinder radius="0.0889" length="0.875"/>
+                <cylinder radius="0.07" length="0.875"/>
             </geometry>
         </visual>
@@ -101,5 +101,5 @@
             <origin rpy="3.14 0 0" xyz="0 0 0.4375"/>
             <geometry>
-                <cylinder radius="0.0889" length="0.875"/>
+                <cylinder radius="0.07" length="0.875"/>
             </geometry>
         </collision>
@@ -134,13 +134,13 @@
     <link name="link3">
         <visual>
-            <origin rpy="1.57079632679 0 0" xyz="0 0.15 0"/>
-            <geometry>
-                <cylinder radius="0.0889" length="0.3"/>
-            </geometry>
-        </visual>
-        <collision>
-            <origin rpy="1.57079632679 0 0" xyz="0 0.15 0"/>
-            <geometry>
-                <cylinder radius="0.0889" length="0.3"/>
+            <origin rpy="1.57079632679 0 0" xyz="0 0.075 0"/>
+            <geometry>
+                <cylinder radius="0.05" length="0.15"/>
+            </geometry>
+        </visual>
+        <collision>
+            <origin rpy="1.57079632679 0 0" xyz="0 0.075 0"/>
+            <geometry>
+                <cylinder radius="0.05" length="0.15"/>
             </geometry>
         </collision>
