Commit message: Remove forearm link

File: uuv_dave/urdf/predator_arm/serial_arm.gazebo.xacro (robot description, xacro)
@@ -28,8 +28,4 @@
     </gazebo>
     <gazebo reference="${namespace}/elbow_link">
-      <selfCollide>false</selfCollide>
-      <maxContacts>1</maxContacts>
-    </gazebo>
-    <gazebo reference="${namespace}/forearm">
       <selfCollide>false</selfCollide>
       <maxContacts>1</maxContacts>
@@ -89,5 +85,4 @@
     <xacro:joint_ft_sensor joint_name="shoulder" namespace="${namespace}"/>
     <xacro:joint_ft_sensor joint_name="elbow" namespace="${namespace}"/>
-    <xacro:joint_ft_sensor joint_name="roll" namespace="${namespace}"/>
     <xacro:joint_ft_sensor joint_name="pitch" namespace="${namespace}"/>
   </xacro:macro>
@@ -146,16 +141,4 @@
       </hydrodynamic_model>
     </link>
-    <link name="${namespace}/forearm">
-      <volume>${total_volume * forearm_volume / total_volume_bbox}</volume>
-      <box>
-        <width>${forearm_width}</width>
-        <length>${forearm_length}</length>
-        <height>${forearm_height}</height>
-      </box>
-      <hydrodynamic_model>
-        <type>cylinder</type>
-        <axis>i</axis>
-      </hydrodynamic_model>
-    </link>
     <link name="${namespace}/wrist_link">
       <volume>${total_volume * wrist_volume / total_volume_bbox}</volume>

File: uuv_dave/urdf/predator_arm/serial_arm.xacro (robot description, xacro)
@@ -107,5 +107,6 @@
             <parent link="${namespace}/shoulder_link"/>
             <child link="${namespace}/upper_arm"/>
-            <origin xyz="0 0 0.1" rpy="${0.5*pi} 0 0"/>
+            <origin xyz="0.1 0 0.1" rpy="${0.5*pi} 0 0"/>
+            <!-- <origin xyz="0 0 0.1" rpy="${0.5*pi} 0 0"/> -->
             <axis xyz="0 0 1"/>
             <!-- <dynamics damping="50" friction="200"/> -->
@@ -147,36 +148,4 @@
         </joint>
         <xacro:simple_transmission joint="${namespace}/elbow" />
-        <!-- FOREARM -->
-        <link name="${namespace}/forearm">
-            <xacro:link_box_inertial mass="${total_mass * forearm_volume / total_volume_bbox}"
-                        width="${forearm_width}"
-                        length="${forearm_length}"
-                        height="${forearm_height}">
-                <origin xyz="${forearm_com}" rpy="0 0 0"/>
-            </xacro:link_box_inertial>
-            <visual>
-                <origin xyz="${forearm_com}" rpy="0 0 0"/>
-                <geometry>
-                    <cylinder radius="${0.5 * forearm_width}" length="${forearm_height}"/>
-                </geometry>
-            </visual>
-            <collision>
-                <origin xyz="${forearm_com}" rpy="0 0 0"/>
-                <geometry>
-                    <cylinder radius="${0.5 * forearm_width}" length="${forearm_height}"/>
-                </geometry>
-            </collision>
-        </link>
-        <joint name="${namespace}/roll" type="revolute">
-            <parent link="${namespace}/elbow_link"/>
-            <child link="${namespace}/forearm"/>
-            <origin xyz="0.1349014 -0.1936267 0" rpy="${0.5*PI} 0 0"/>
-            <axis xyz="0 0 1"/>
-            <!-- <dynamics damping="50" friction="200"/> -->
-            <dynamics damping="300" friction="1000"/>
-            <!-- <limit lower="${-135 * d2r}" upper="${135 * d2r}" velocity=".15" effort="200"/> -->
-            <limit lower="${-135 * d2r}" upper="${135 * d2r}" velocity=".25" effort="1000"/>
-        </joint>
-        <xacro:simple_transmission joint="${namespace}/roll" />
         <!-- WRIST 1  -->
         <link name="${namespace}/wrist_link">
@@ -201,7 +170,7 @@
         </link>
         <joint name="${namespace}/pitch" type="revolute">
-            <parent link="${namespace}/forearm"/>
+            <parent link="${namespace}/elbow_link"/>
             <child link="${namespace}/wrist_link"/>
-            <origin xyz="0 0 0.31595760629823427" rpy="${-0.5*PI} ${-0.5*PI} 0"/>
+            <origin xyz="${0.1349014*3} ${-0.1936267-0.31595760629823427} 0" rpy="${-0*PI} ${-0*PI} 0"/>
             <axis xyz="0 0 1"/>
             <!-- <dynamics damping="50" friction="200"/> -->
