Commit message: Convert most of links to cylinders

File: uuv_dave/urdf/predator_arm/serial_arm.xacro (robot description, xacro)
@@ -51,15 +51,10 @@
             </xacro:link_box_inertial>
             <visual>
-                <origin xyz="0 0 0" rpy="0 0 0"/>
-                <geometry>
-                    <mesh filename="file://$(find oberon7_description)/meshes/serial_arm/visual/Base.dae"/>
-                </geometry>
-            </visual>
-            <collision>
-                <origin xyz="0 0 0" rpy="0 0 0"/>
-                <geometry>
-                    <mesh filename="file://$(find oberon7_description)/meshes/serial_arm/collision/Base.stl"/>
-                </geometry>
-            </collision>
+                <origin xyz="0 0 -0.09" rpy="0 0 0"/>
+                <geometry>
+                    <!-- <box size="0.197 0.197 0.04524"/> -->
+                    <box size="0.197 0.197 0.04524"/>
+                </geometry>
+            </visual>
         </link>
         <!-- Shoulder link -->
@@ -74,13 +69,7 @@
                 <origin xyz="0 0 0" rpy="0 0 0"/>
                 <geometry>
-                    <mesh filename="file://$(find oberon7_description)/meshes/serial_arm/visual/ShoulderLink.dae"/>
-                </geometry>
-            </visual>
-            <collision>
-                <origin xyz="${shoulder_link_com}" rpy="0 0 0"/>
-                <geometry>
-                    <cylinder radius="${0.5 * shoulder_link_width}" length="${shoulder_link_height}" />
-                </geometry>
-            </collision>
+                    <cylinder radius="${0.0985}" length="0.15776" />
+                </geometry>
+            </visual>
         </link>
         <joint name="${namespace}/azimuth" type="revolute">
@@ -103,11 +92,11 @@
             </xacro:link_box_inertial>
             <visual>
-                <origin xyz="0 0 0" rpy="0 0 0"/>
-                <geometry>
-                    <mesh filename="file://$(find oberon7_description)/meshes/serial_arm/visual/UpperArm.dae"/>
-                </geometry>
-            </visual>
-            <collision>
-                <origin xyz="${upper_arm_com}" rpy="0 ${0.5*pi} 0"/>
+                <origin xyz="0.312501 0 0" rpy="0 ${0.5*pi} 0"/>
+                <geometry>
+                    <cylinder radius="${0.5 * upper_arm_width}" length="${upper_arm_length}"/>
+                </geometry>
+            </visual>
+            <collision>
+                <origin xyz="0.312501 0 0" rpy="0 ${0.5*pi} 0"/>
                 <geometry>
                     <cylinder radius="${0.5 * upper_arm_width}" length="${upper_arm_length}"/>
@@ -118,5 +107,5 @@
             <parent link="${namespace}/shoulder_link"/>
             <child link="${namespace}/upper_arm"/>
-            <origin xyz="0.06955 0.00015 0.01536" rpy="${0.5*pi} 0 0"/>
+            <origin xyz="0 0 0.1" rpy="${0.5*pi} 0 0"/>
             <axis xyz="0 0 1"/>
             <!-- <dynamics damping="50" friction="200"/> -->
@@ -135,13 +124,13 @@
             </xacro:link_box_inertial>
             <visual>
-                <origin xyz="0 0 0" rpy="0 0 0"/>
-                <geometry>
-                    <mesh filename="file://$(find oberon7_description)/meshes/serial_arm/visual/ElbowLink.dae"/>
-                </geometry>
-            </visual>
-            <collision>
-                <origin xyz="${elbow_link_com}" rpy="0 ${0.5*pi} ${0.5*pi}"/>
-                <geometry>
-                    <cylinder radius="${0.5 * elbow_link_height}" length="${elbow_link_length}"/>
+                <origin xyz="0.125269 ${-elbow_link_length/2-forearm_height/2} 0.0" rpy="0 ${0.5*pi} ${0.5*pi}"/>
+                <geometry>
+                    <cylinder radius="${0.5 * elbow_link_height}" length="${elbow_link_length+forearm_height}"/>
+                </geometry>
+            </visual>
+            <collision>
+                <origin xyz="0.125269 ${-elbow_link_length/2-forearm_height/2} 0.0" rpy="0 ${0.5*pi} ${0.5*pi}"/>
+                <geometry>
+                    <cylinder radius="${0.5 * elbow_link_height}" length="${elbow_link_length+forearm_height}"/>
                 </geometry>
             </collision>
@@ -167,7 +156,7 @@
             </xacro:link_box_inertial>
             <visual>
-                <origin xyz="0 0 0" rpy="0 0 0"/>
-                <geometry>
-                    <mesh filename="file://$(find oberon7_description)/meshes/serial_arm/visual/Forearm.dae"/>
+                <origin xyz="${forearm_com}" rpy="0 0 0"/>
+                <geometry>
+                    <cylinder radius="${0.5 * forearm_width}" length="${forearm_height}"/>
                 </geometry>
             </visual>

File: uuv_dave/urdf/rexrov_predator.xacro (robot description, xacro)
@@ -74,5 +74,5 @@
   </xacro:rexrov_base>
   <xacro:oberon7 namespace="oberon7" parent="$(arg namespace)/base_link">
-    <origin xyz="1.3 -0.5 -0.615" rpy="0 0 0"/>
+    <origin xyz="1 -0.5 -0.615" rpy="0 0 0"/>
   </xacro:oberon7>
   <gazebo>

Commit message: Correct joint locations for first 3 links

File: uuv_dave/urdf/predator_arm/serial_arm.xacro (robot description, xacro)
@@ -48,15 +48,15 @@
                         length="${base_length}"
                         height="${base_height}">
-            <origin xyz="${base_com}" rpy="0 0 0"/>
+            <origin xyz="0 0 0" rpy="0 0 0"/>
             </xacro:link_box_inertial>
-            <visual>
-                <origin xyz="0 0 -0.09" rpy="0 0 0"/>
+            <!-- <visual>
+                <origin xyz="0 0 ${-0.15776/2+0.015776/2}" rpy="0 0 0"/>
                 <geometry>
-                    <!-- <box size="0.197 0.197 0.04524"/> -->
-                    <box size="0.197 0.197 0.04524"/>
+                    <box size="0.197 0.197 0.015776"/>
                 </geometry>
-            </visual>
+            </visual> -->
         </link>
         <!-- Shoulder link -->
+        <xacro:property name="base_height" value="0.203"/>
         <link name="${namespace}/shoulder_link">
             <xacro:link_box_inertial mass="${total_mass * shoulder_link_volume / total_volume_bbox}"
@@ -67,11 +67,12 @@
             </xacro:link_box_inertial>
             <visual>
-                <origin xyz="0 0 0" rpy="0 0 0"/>
+                <origin xyz="0 0 ${-base_height/2}" rpy="0 0 0"/>
                 <geometry>
-                    <cylinder radius="${0.0985}" length="0.15776" />
+                    <cylinder radius="${0.0985}" length="${base_height}" />
                 </geometry>
             </visual>
         </link>
         <joint name="${namespace}/azimuth" type="revolute">
+            <origin xyz="0 0 ${0.203/2}" rpy="0 0 0"/>
             <parent link="${namespace}/base"/>
             <child link="${namespace}/shoulder_link"/>
@@ -84,4 +85,5 @@
         <xacro:simple_transmission joint="${namespace}/azimuth" />
         <!-- UPPER ARM -->
+        <xacro:property name="upper_arm_l" value="${0.939}"/>
         <link name="${namespace}/upper_arm">
             <xacro:link_box_inertial mass="${total_mass * upper_arm_volume / total_volume_bbox}"
@@ -92,20 +94,20 @@
             </xacro:link_box_inertial>
             <visual>
+                <origin xyz="${upper_arm_l/2} 0 0" rpy="0 ${0.5*pi} 0"/>
+                <geometry>
+                    <cylinder radius="${0.5 * upper_arm_width}" length="${upper_arm_l}"/>
+                </geometry>
+            </visual>
+            <!-- <collision>
                 <origin xyz="0.312501 0 0" rpy="0 ${0.5*pi} 0"/>
                 <geometry>
-                    <cylinder radius="${0.5 * upper_arm_width}" length="${upper_arm_length}"/>
+                    <cylinder radius="${0.5 * upper_arm_width}" length="${upper_arm_length+.34712}"/>
                 </geometry>
-            </visual>
-            <collision>
-                <origin xyz="0.312501 0 0" rpy="0 ${0.5*pi} 0"/>
-                <geometry>
-                    <cylinder radius="${0.5 * upper_arm_width}" length="${upper_arm_length}"/>
-                </geometry>
-            </collision>
+            </collision> -->
         </link>
         <joint name="${namespace}/shoulder" type="revolute">
             <parent link="${namespace}/shoulder_link"/>
             <child link="${namespace}/upper_arm"/>
-            <origin xyz="0.1 0 0.1" rpy="${0.5*pi} 0 0"/>
+            <origin xyz="0.1 0 0" rpy="${0.5*pi} 0 0"/>
             <!-- <origin xyz="0 0 0.1" rpy="${0.5*pi} 0 0"/> -->
             <axis xyz="0 0 1"/>
@@ -126,4 +128,5 @@
             <visual>
                 <origin xyz="0.125269 ${-elbow_link_length/2-forearm_height/2} 0.0" rpy="0 ${0.5*pi} ${0.5*pi}"/>
+                <!-- <origin xyz="0.125269 ${-forearm_height/2} 0.0" rpy="0 ${0.5*pi} ${0.5*pi}"/> -->
                 <geometry>
                     <cylinder radius="${0.5 * elbow_link_height}" length="${elbow_link_length+forearm_height}"/>
@@ -133,5 +136,5 @@
                 <origin xyz="0.125269 ${-elbow_link_length/2-forearm_height/2} 0.0" rpy="0 ${0.5*pi} ${0.5*pi}"/>
                 <geometry>
-                    <cylinder radius="${0.5 * elbow_link_height}" length="${elbow_link_length+forearm_height}"/>
+                    <cylinder radius="${0.5 * elbow_link_height}" length="${elbow_link_length/3+forearm_height/3}"/>
                 </geometry>
             </collision>
@@ -140,5 +143,5 @@
             <parent link="${namespace}/upper_arm"/>
             <child link="${namespace}/elbow_link"/>
-            <origin xyz="0.55616 -0.01229 0" rpy="0 0 0"/>
+            <origin xyz="${upper_arm_l-0.064} 0 0" rpy="0 0 0"/>
             <!-- <dynamics damping="50" friction="200"/> -->
             <dynamics damping="50" friction="150"/>
@@ -172,5 +175,7 @@
             <parent link="${namespace}/elbow_link"/>
             <child link="${namespace}/wrist_link"/>
-            <origin xyz="${0.1349014*3} ${-0.1936267-0.31595760629823427} 0" rpy="${-0*PI} ${-0*PI} 0"/>
+            <!-- <origin xyz="${0.210} ${-0.525} 0" rpy="0 0 ${-0.5*PI}"/> -->
+            <!-- <origin xyz="${0.1349014} ${-0.1936267/3-0.31595760629823427/3} 0" rpy="${-0*PI} ${-0*PI} ${-0.5*PI}"/> -->
+            <origin xyz="${0.1349014} ${-0.1936267/3-0.31595760629823427/3} 0" rpy="${-0*PI} ${-0*PI} ${-0.5*PI}"/>
             <axis xyz="0 0 1"/>
             <!-- <dynamics damping="50" friction="200"/> -->

File: uuv_dave/urdf/rexrov_predator.xacro (robot description, xacro)
@@ -74,5 +74,5 @@
   </xacro:rexrov_base>
   <xacro:oberon7 namespace="oberon7" parent="$(arg namespace)/base_link">
-    <origin xyz="1 -0.5 -0.615" rpy="0 0 0"/>
+    <origin xyz="1.2 -0.5 -0.595" rpy="0 0 0"/>
   </xacro:oberon7>
   <gazebo>
